File: arduino-day-arduino.brd (EAGLE design)
At the start: 84.8 x 54.6 mm, 27 parts, among them Q2 16Mhz, X2 USB-B_TH

Commit message: Board routed
Parts:
- moved SJ2 1.27 mm to (31.8, 35.6)
- moved SJ1 1.27 mm to (26.7, 35.6)
Routing:
- net +5V: track 0.00 -> 165.5 mm
- net SDA: track 0.00 -> 100.4 mm, vias 0 -> 1
- net SCL: track 0.00 -> 97.5 mm, vias 0 -> 1
- net MISO: track 0.00 -> 82.1 mm, vias 0 -> 1
- net TX: track 0.00 -> 77.3 mm, vias 0 -> 1
- net SCK: track 0.00 -> 76.0 mm, vias 0 -> 1
- net RX: track 0.00 -> 75.8 mm, vias 0 -> 1
- net MOSI: track 0.00 -> 73.4 mm, vias 0 -> 2
- net AREF: track 0.00 -> 68.6 mm
- net +3V3: track 0.00 -> 62.4 mm, vias 0 -> 1
- net RST: track 0.00 -> 58.4 mm, vias 0 -> 1
- net N$15: track 0.00 -> 54.0 mm, vias 0 -> 1
- net N$16: track 0.00 -> 48.9 mm, vias 0 -> 1
- net N$6: track 0.00 -> 48.5 mm, vias 0 -> 1
- net USB-SDA: track 0.00 -> 47.9 mm
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- added copper zone on layer 1, net GND
- added copper zone on layer 16, net GND

Commit message: Logok
Parts:
- added C5: 22pF, rcl:C025-025X050
- renumbered D0-D7 to D, SV1 to PWR
Connections:
- net AREF: now also C5.1
- net GND: now also C5.2
Routing:
- net AREF: track 68.6 -> 76.8 mm
- net N$16: track 48.9 -> 50.0 mm
Other:
- board text added: "+3V3"
- board text added: "+5V"
- board text added: "A0"
- board text added: "A1"
- board text added: "A2"
- board text added: "A3"
- board text added: "A4"
- board text added: "A5"
- board text added: "AREF"
- board text added: "CsharptutorialHungary/diydunio"
- board text added: "D0"
- board text added: "D1"
- board text added: "D10"
- board text added: "D11"
- board text added: "D12"
- board text added: "D13"
- board text added: "D2"
- board text added: "D3"
- board text added: "D4"
- board text added: "D5"
- board text added: "D6"
- board text added: "D7"
- board text added: "D8"
- board text added: "D9"
- board text added: "DIYDunio V1"
- board text added: "GND"
- board text added: "RST"
- board text added: "SCL"
- board text added: "SDA"

Commit message: Orderable
Parts:
- renumbered SJ1 to U-SCL-5V, SJ2 to U-SDA-5V
Changed lines of the file:
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@@
 <grid distance="12" unitdist="mil" unit="mil" style="lines" multiple="1" display="no" altdistance="5" altunitdist="mil" altunit="mil"/>
 <layers>
-<layer number="1" name="Top" color="4" fill="1" visible="yes" active="yes"/>
+<layer number="1" name="Top" color="4" fill="1" visible="no" active="yes"/>
 <layer number="2" name="Route2" color="16" fill="1" visible="no" active="no"/>
 <layer number="3" name="Route3" color="17" fill="1" visible="no" active="no"/>
@@
 <layer number="14" name="Route14" color="22" fill="1" visible="no" active="no"/>
 <layer number="15" name="Route15" color="23" fill="1" visible="no" active="no"/>
-<layer number="16" name="Bottom" color="1" fill="1" visible="yes" active="yes"/>
+<layer number="16" name="Bottom" color="1" fill="1" visible="no" active="yes"/>
 <layer number="17" name="Pads" color="2" fill="1" visible="yes" active="yes"/>
 <layer number="18" name="Vias" color="2" fill="1" visible="yes" active="yes"/>
 <layer number="19" name="Unrouted" color="6" fill="1" visible="yes" active="yes"/>
 <layer number="20" name="Dimension" color="24" fill="1" visible="yes" active="yes"/>
-<layer number="21" name="tPlace" color="7" fill="1" visible="no" active="yes"/>
-<layer number="22" name="bPlace" color="7" fill="1" visible="yes" active="yes"/>
+<layer number="21" name="tPlace" color="7" fill="1" visible="yes" active="yes"/>
+<layer number="22" name="bPlace" color="7" fill="1" visible="no" active="yes"/>
 <layer number="23" name="tOrigins" color="15" fill="1" visible="yes" active="yes"/>
 <layer number="24" name="bOrigins" color="15" fill="1" visible="yes" active="yes"/>
@@
 <element name="3V3REG" library="adafruit" package="TO92" value="MCP1700-3302E/TO" x="11.43" y="43.18" smashed="yes" rot="R270">
 <attribute name="NAME" x="13.081" y="40.767" size="1.27" layer="25" ratio="10" rot="R270"/>
-<attribute name="VALUE" x="7.62" y="49.149" size="1.27" layer="27" ratio="10" rot="R270"/>
+<attribute name="VALUE" x="8.2296" y="47.3202" size="1.27" layer="27" ratio="10" rot="R270"/>
 </element>
 <element name="A0-A5" library="con-lsta" library_urn="urn:adsk.eagle:library:161" package="FE06" package3d_urn="urn:adsk.eagle:package:8191/1" value="" x="80.01" y="12.7" smashed="yes">
@@
 </element>
 <element name="MCU" library="SmartPrj" package="DIL28-3" value="ATMEGA328P-PU" x="60.96" y="26.67" smashed="yes" rot="R180">
-<attribute name="NAME" x="80.1624" y="29.21" size="1.778" layer="25" ratio="10" rot="R270"/>
-<attribute name="VALUE" x="76.835" y="27.305" size="1.778" layer="27" ratio="10" rot="R180"/>
+<attribute name="NAME" x="77.978" y="28.0416" size="1.778" layer="25" ratio="10" rot="R180"/>
+<attribute name="VALUE" x="66.7766" y="26.6954" size="1.778" layer="27" ratio="10" rot="R180"/>
 </element>
 <element name="Q2" library="crystal" package="HC49/S" value="16Mhz" x="55.88" y="36.83" smashed="yes">
@@
 <attribute name="VALUE" x="16.9926" y="26.3144" size="0.9906" layer="27" ratio="10" rot="R90"/>
 </element>
-<element name="SJ1" library="jumper" library_urn="urn:adsk.eagle:library:252" package="SJW" package3d_urn="urn:adsk.eagle:package:15507/1" value="" x="26.67" y="35.56" smashed="yes" rot="R90">
-<attribute name="NAME" x="24.892" y="33.401" size="1.27" layer="25" ratio="10" rot="R90"/>
+<element name="U-SCL-5V" library="jumper" library_urn="urn:adsk.eagle:library:252" package="SJW" package3d_urn="urn:adsk.eagle:package:15507/1" value="" x="26.67" y="35.56" smashed="yes" rot="R90">
+<attribute name="NAME" x="24.892" y="31.877" size="1.27" layer="25" ratio="10" rot="R90"/>
 <attribute name="POPULARITY" value="3" x="113.03" y="80.01" size="1.778" layer="27" rot="R90" display="off"/>
 <attribute name="VALUE" x="26.67" y="36.56" size="0.02" layer="27" rot="R90"/>
 </element>
-<element name="SJ2" library="jumper" library_urn="urn:adsk.eagle:library:252" package="SJW" package3d_urn="urn:adsk.eagle:package:15507/1" value="" x="31.75" y="35.56" smashed="yes" rot="R90">
-<attribute name="NAME" x="29.972" y="33.401" size="1.27" layer="25" ratio="10" rot="R90"/>
+<element name="U-SDA-5V" library="jumper" library_urn="urn:adsk.eagle:library:252" package="SJW" package3d_urn="urn:adsk.eagle:package:15507/1" value="" x="31.75" y="35.56" smashed="yes" rot="R90">
+<attribute name="NAME" x="34.8488" y="31.5722" size="1.27" layer="25" ratio="10" rot="R90"/>
 <attribute name="POPULARITY" value="3" x="118.11" y="85.09" size="1.778" layer="27" rot="R90" display="off"/>
 <attribute name="VALUE" x="31.75" y="36.56" size="0.02" layer="27" rot="R90"/>
@@
 </element>
 <element name="USBSERIAL" library="Webmaster442" package="DIL14" value="MCP2221" x="31.75" y="49.53" smashed="yes" rot="R90">
-<attribute name="NAME" x="34.798" y="40.259" size="1.27" layer="25" ratio="10" rot="R180"/>
+<attribute name="NAME" x="32.5882" y="51.8668" size="1.27" layer="25" ratio="10" rot="R270"/>
 <attribute name="VALUE" x="32.385" y="42.799" size="1.27" layer="27" ratio="10" rot="R90"/>
 </element>
@@
 <contactref element="R1" pad="1"/>
 <contactref element="ISP1" pad="2"/>
-<contactref element="SJ2" pad="2"/>
-<contactref element="SJ1" pad="2"/>
+<contactref element="U-SDA-5V" pad="2"/>
+<contactref element="U-SCL-5V" pad="2"/>
 <contactref element="USB-I2C" pad="2"/>
 <contactref element="I2C" pad="2"/>
@@
 <signal name="N$17">
 <contactref element="R2" pad="2"/>
-<contactref element="SJ2" pad="1"/>
+<contactref element="U-SDA-5V" pad="1"/>
 <wire x1="31.75" y1="34.29" x2="33.02" y2="34.29" width="0.254" layer="1"/>
 <wire x1="33.02" y1="34.29" x2="34.29" y2="33.02" width="0.254" layer="1"/>
@@
 </signal>
 <signal name="N$18">
-<contactref element="SJ1" pad="1"/>
+<contactref element="U-SCL-5V" pad="1"/>
 <contactref element="R3" pad="2"/>
 <wire x1="26.67" y1="34.29" x2="29.21" y2="31.75" width="0.254" layer="1"/>
