File: arduino-day-arduino.sch (EAGLE design)
At the start: 28 parts, among them Q2 16Mhz, X2 USB-B_TH

Commit message: Board layout
Parts:
- removed AREF-RST: (no value), con-lstb:MA03-1
- removed D8-D13: (no value), con-lsta:FE06-1
- removed PWR: (no value), con-lstb:MA06-1
- added SV1: (no value), con-lsta:FE08-1
- added SV2: (no value), con-lsta:FE10-1
- C1, C2: value 1uf -> 1uF
- C3, C4: device rcl:C-EU025-060X050 -> rcl:C-EU025-025X050
- R4, R5, R6: device rcl:R-EU_R1206 -> rcl:R-EU_0204/7
Connections:
- net +3V3: now also SV1.5; no longer PWR.5, PWR.6
- net +5V: now also SV1.4; no longer PWR.1, PWR.2
- net AREF: now also SV1.7, SV2.8; no longer AREF-RST.2
- net GND: now also SV1.2, SV1.3, SV2.7; no longer AREF-RST.1, PWR.3, PWR.4
- net LED_RX: now also R4.2; no longer R4.1
- net LED_TX: now also R5.2; no longer R5.1
- net MISO: now also SV2.5; no longer D8-D13.5
- net MOSI: now also SV2.4; no longer D8-D13.4
- net N$14: now also SV2.1; no longer D8-D13.1
- net N$15: now also SV2.2; no longer D8-D13.2
- net N$16: now also SV2.3; no longer D8-D13.3
- net N$28: now also R4.1; no longer R4.2
- net N$29: now also R5.1; no longer R5.2
- net N$30: now also R6.1; no longer R6.2
- net N$31: now also R6.2; no longer R6.1
- net N$37: now also C3.2; no longer C4.2
- net N$38: now also C4.2; no longer C3.2
- net RST: now also SV1.6; no longer AREF-RST.3
- net SCK: now also SV2.6; no longer D8-D13.6
- net SCL: now also SV2.10
- net SDA: now also SV2.9
Other:
- moved on the sheet: C3, C4, I2C, R4, R5, R6, USB-I2C

Commit message: Logok
Parts:
- added C5: 22pF, rcl:C-EU025-025X050
- renumbered D0-D7 to D, SV1 to PWR
Connections:
- net AREF: now also C5.1
- net GND: now also C5.2
Changed lines of the file:
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@@
 <part name="GND4" library="supply1" deviceset="GND" device=""/>
 <part name="A0-A5" library="con-lsta" library_urn="urn:adsk.eagle:library:161" deviceset="FE06-1" device="" package3d_urn="urn:adsk.eagle:package:8191/1"/>
-<part name="D0-D7" library="con-lsta" library_urn="urn:adsk.eagle:library:161" deviceset="FE08-1" device="" package3d_urn="urn:adsk.eagle:package:8194/1"/>
+<part name="D" library="con-lsta" library_urn="urn:adsk.eagle:library:161" deviceset="FE08-1" device="" package3d_urn="urn:adsk.eagle:package:8194/1"/>
 <part name="R2" library="rcl" deviceset="R-EU_" device="0204/7" value="10k"/>
 <part name="R3" library="rcl" deviceset="R-EU_" device="0204/7" value="10k"/>
@@
 <part name="C3" library="rcl" library_urn="urn:adsk.eagle:library:334" deviceset="C-EU" device="025-025X050" package3d_urn="urn:adsk.eagle:package:23629/2" value="22pF"/>
 <part name="C4" library="rcl" library_urn="urn:adsk.eagle:library:334" deviceset="C-EU" device="025-025X050" package3d_urn="urn:adsk.eagle:package:23629/2" value="22pF"/>
-<part name="SV1" library="con-lsta" library_urn="urn:adsk.eagle:library:161" deviceset="FE08-1" device="" package3d_urn="urn:adsk.eagle:package:8194/1"/>
+<part name="PWR" library="con-lsta" library_urn="urn:adsk.eagle:library:161" deviceset="FE08-1" device="" package3d_urn="urn:adsk.eagle:package:8194/1"/>
 <part name="GND6" library="supply1" deviceset="GND" device=""/>
 <part name="+3V2" library="supply1" library_urn="urn:adsk.eagle:library:371" deviceset="+3V3" device=""/>
@@
 <part name="SV2" library="con-lsta" library_urn="urn:adsk.eagle:library:161" deviceset="FE10-1" device="" package3d_urn="urn:adsk.eagle:package:8192/1"/>
 <part name="GND7" library="supply1" deviceset="GND" device=""/>
+<part name="C5" library="rcl" library_urn="urn:adsk.eagle:library:334" deviceset="C-EU" device="025-025X050" package3d_urn="urn:adsk.eagle:package:23629/2" value="22pF"/>
+<part name="GND8" library="supply1" deviceset="GND" device=""/>
 </parts>
 <sheets>
@@
 <attribute name="NAME" x="146.05" y="64.262" size="1.778" layer="95" rot="MR0"/>
 </instance>
-<instance part="D0-D7" gate="G$1" x="137.16" y="33.02" smashed="yes" rot="MR0">
+<instance part="D" gate="G$1" x="137.16" y="33.02" smashed="yes" rot="MR0">
 <attribute name="VALUE" x="138.43" y="20.32" size="1.778" layer="96" rot="MR0"/>
 <attribute name="NAME" x="138.43" y="46.482" size="1.778" layer="95" rot="MR0"/>
@@
 <attribute name="VALUE" x="52.959" y="62.484" size="1.778" layer="96" rot="R90"/>
 </instance>
-<instance part="SV1" gate="G$1" x="40.64" y="-10.16" smashed="yes">
+<instance part="PWR" gate="G$1" x="40.64" y="-10.16" smashed="yes">
 <attribute name="VALUE" x="39.37" y="-22.86" size="1.778" layer="96"/>
 <attribute name="NAME" x="39.37" y="3.302" size="1.778" layer="95"/>
@@
 <instance part="GND7" gate="1" x="127" y="15.24" smashed="yes">
 <attribute name="VALUE" x="124.46" y="12.7" size="1.778" layer="96"/>
+</instance>
+<instance part="C5" gate="G$1" x="50.8" y="40.64" smashed="yes">
+<attribute name="NAME" x="52.324" y="41.021" size="1.778" layer="95"/>
+<attribute name="VALUE" x="52.324" y="35.941" size="1.778" layer="96"/>
+</instance>
+<instance part="GND8" gate="1" x="50.8" y="30.48" smashed="yes">
+<attribute name="VALUE" x="48.26" y="27.94" size="1.778" layer="96"/>
 </instance>
 </instances>
@@
 </segment>
 <segment>
-<pinref part="SV1" gate="G$1" pin="4"/>
+<pinref part="PWR" gate="G$1" pin="4"/>
 <wire x1="48.26" y1="-10.16" x2="53.34" y2="-10.16" width="0.1524" layer="91"/>
 <wire x1="53.34" y1="-10.16" x2="53.34" y2="7.62" width="0.1524" layer="91"/>
@@
 </segment>
 <segment>
-<pinref part="SV1" gate="G$1" pin="2"/>
+<pinref part="PWR" gate="G$1" pin="2"/>
 <wire x1="48.26" y1="-15.24" x2="53.34" y2="-15.24" width="0.1524" layer="91"/>
 <wire x1="53.34" y1="-15.24" x2="53.34" y2="-12.7" width="0.1524" layer="91"/>
-<pinref part="SV1" gate="G$1" pin="3"/>
+<pinref part="PWR" gate="G$1" pin="3"/>
 <wire x1="53.34" y1="-12.7" x2="48.26" y2="-12.7" width="0.1524" layer="91"/>
 <wire x1="53.34" y1="-15.24" x2="53.34" y2="-20.32" width="0.1524" layer="91"/>
@@
 <pinref part="GND7" gate="1" pin="GND"/>
 </segment>
+<segment>
+<pinref part="C5" gate="G$1" pin="2"/>
+<pinref part="GND8" gate="1" pin="GND"/>
+<wire x1="50.8" y1="35.56" x2="50.8" y2="33.02" width="0.1524" layer="91"/>
+</segment>
 </net>
 <net name="TX" class="0">
@@
 <wire x1="129.54" y1="25.4" x2="119.38" y2="25.4" width="0.1524" layer="91"/>
 <label x="119.38" y="25.4" size="1.778" layer="95"/>
-<pinref part="D0-D7" gate="G$1" pin="1"/>
+<pinref part="D" gate="G$1" pin="1"/>
 <junction x="129.54" y="25.4"/>
 <wire x1="129.54" y1="25.4" x2="116.84" y2="25.4" width="0.1524" layer="91"/>
@@
 <wire x1="119.38" y1="27.94" x2="129.54" y2="27.94" width="0.1524" layer="91"/>
 <label x="119.38" y="27.94" size="1.778" layer="95"/>
-<pinref part="D0-D7" gate="G$1" pin="2"/>
+<pinref part="D" gate="G$1" pin="2"/>
 <junction x="129.54" y="27.94"/>
 <wire x1="129.54" y1="27.94" x2="116.84" y2="27.94" width="0.1524" layer="91"/>
@@
 </segment>
 <segment>
-<pinref part="SV1" gate="G$1" pin="6"/>
+<pinref part="PWR" gate="G$1" pin="6"/>
 <wire x1="48.26" y1="-5.08" x2="66.04" y2="-5.08" width="0.1524" layer="91"/>
 <label x="66.04" y="-5.08" size="1.778" layer="95"/>
@@
 </segment>
 <segment>
-<pinref part="SV1" gate="G$1" pin="5"/>
+<pinref part="PWR" gate="G$1" pin="5"/>
 <wire x1="48.26" y1="-7.62" x2="60.96" y2="-7.62" width="0.1524" layer="91"/>
 <wire x1="60.96" y1="-7.62" x2="60.96" y2="5.08" width="0.1524" layer="91"/>
@@
 <segment>
 <pinref part="MCU" gate="G$1" pin="(INT0)PD2"/>
-<pinref part="D0-D7" gate="G$1" pin="3"/>
+<pinref part="D" gate="G$1" pin="3"/>
 <wire x1="129.54" y1="30.48" x2="116.84" y2="30.48" width="0.1524" layer="91"/>
 </segment>
@@
 <segment>
 <pinref part="MCU" gate="G$1" pin="(INT1)PD3"/>
-<pinref part="D0-D7" gate="G$1" pin="4"/>
+<pinref part="D" gate="G$1" pin="4"/>
 <wire x1="129.54" y1="33.02" x2="116.84" y2="33.02" width="0.1524" layer="91"/>
 </segment>
@@
 <segment>
 <pinref part="MCU" gate="G$1" pin="(T0)PD4"/>
-<pinref part="D0-D7" gate="G$1" pin="5"/>
+<pinref part="D" gate="G$1" pin="5"/>
 <wire x1="129.54" y1="35.56" x2="116.84" y2="35.56" width="0.1524" layer="91"/>
 </segment>
@@
 <segment>
 <pinref part="MCU" gate="G$1" pin="(T1)PD5"/>
-<pinref part="D0-D7" gate="G$1" pin="6"/>
+<pinref part="D" gate="G$1" pin="6"/>
 <wire x1="129.54" y1="38.1" x2="116.84" y2="38.1" width="0.1524" layer="91"/>
 </segment>
@@
 <segment>
 <pinref part="MCU" gate="G$1" pin="(AIN0)PD6"/>
-<pinref part="D0-D7" gate="G$1" pin="7"/>
+<pinref part="D" gate="G$1" pin="7"/>
 <wire x1="129.54" y1="40.64" x2="116.84" y2="40.64" width="0.1524" layer="91"/>
 </segment>
@@
 <segment>
 <pinref part="MCU" gate="G$1" pin="(AIN1)PD7"/>
-<pinref part="D0-D7" gate="G$1" pin="8"/>
+<pinref part="D" gate="G$1" pin="8"/>
 <wire x1="129.54" y1="43.18" x2="116.84" y2="43.18" width="0.1524" layer="91"/>
 </segment>
@@
 </segment>
 <segment>
-<pinref part="SV1" gate="G$1" pin="7"/>
+<pinref part="PWR" gate="G$1" pin="7"/>
 <wire x1="48.26" y1="-2.54" x2="66.04" y2="-2.54" width="0.1524" layer="91"/>
 <label x="66.04" y="-2.54" size="1.778" layer="95"/>
@@
 <label x="114.3" y="83.82" size="1.778" layer="95"/>
 </segment>
-</net>
+<segment>
+<pinref part="C5" gate="G$1" pin="1"/>
+<wire x1="50.8" y1="43.18" x2="50.8" y2="48.26" width="0.1524" layer="91"/>
+<wire x1="50.8" y1="48.26" x2="45.72" y2="48.26" width="0.1524" layer="91"/>
+<label x="40.64" y="48.26" size="1.778" layer="95"/>
+</segment>
+</net>

Commit message: Orderable
Parts:
- renumbered SJ1 to U-SCL-5V, SJ2 to U-SDA-5V
Other:
- note removed: "Projekt felmásolása"
Changed lines of the file:
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@@
 <part name="L3" library="led" library_urn="urn:adsk.eagle:library:259" deviceset="LED" device="3MM" package3d_urn="urn:adsk.eagle:package:15797/1"/>
 <part name="P+15" library="supply1" library_urn="urn:adsk.eagle:library:371" deviceset="+5V" device=""/>
-<part name="SJ2" library="jumper" library_urn="urn:adsk.eagle:library:252" deviceset="SJ" device="W" package3d_urn="urn:adsk.eagle:package:15507/1"/>
+<part name="U-SDA-5V" library="jumper" library_urn="urn:adsk.eagle:library:252" deviceset="SJ" device="W" package3d_urn="urn:adsk.eagle:package:15507/1"/>
 <part name="MCU" library="SmartPrj" deviceset="ATMEGA328P-" device="PU"/>
 <part name="Q2" library="crystal" deviceset="CRYSTAL" device="HC49S" value="16Mhz"/>
@@
 <part name="R2" library="rcl" deviceset="R-EU_" device="0204/7" value="10k"/>
 <part name="R3" library="rcl" deviceset="R-EU_" device="0204/7" value="10k"/>
-<part name="SJ1" library="jumper" library_urn="urn:adsk.eagle:library:252" deviceset="SJ" device="W" package3d_urn="urn:adsk.eagle:package:15507/1"/>
+<part name="U-SCL-5V" library="jumper" library_urn="urn:adsk.eagle:library:252" deviceset="SJ" device="W" package3d_urn="urn:adsk.eagle:package:15507/1"/>
 <part name="USB-I2C" library="con-lstb" library_urn="urn:adsk.eagle:library:162" deviceset="MA04-1" device="" package3d_urn="urn:adsk.eagle:package:8337/1"/>
 <part name="I2C" library="con-lstb" library_urn="urn:adsk.eagle:library:162" deviceset="MA04-1" device="" package3d_urn="urn:adsk.eagle:package:8337/1"/>
@@
 <sheet>
 <plain>
-<text x="-48.26" y="-2.54" size="1.778" layer="91">Projekt felmásolása</text>
 </plain>
 <instances>
@@
 <attribute name="VALUE" x="-53.34" y="76.2" size="1.778" layer="96" rot="R90"/>
 </instance>
-<instance part="SJ2" gate="1" x="2.54" y="83.82" smashed="yes" rot="R90">
+<instance part="U-SDA-5V" gate="1" x="2.54" y="83.82" smashed="yes" rot="R90">
 <attribute name="NAME" x="0" y="81.28" size="1.778" layer="95" rot="R90"/>
 <attribute name="VALUE" x="6.35" y="81.28" size="1.778" layer="96" rot="R90"/>
@@
 <attribute name="VALUE" x="13.462" y="67.31" size="1.778" layer="96" rot="R90"/>
 </instance>
-<instance part="SJ1" gate="1" x="10.16" y="83.82" smashed="yes" rot="R90">
+<instance part="U-SCL-5V" gate="1" x="10.16" y="83.82" smashed="yes" rot="R90">
 <attribute name="NAME" x="7.62" y="81.28" size="1.778" layer="95" rot="R90"/>
 <attribute name="VALUE" x="13.97" y="81.28" size="1.778" layer="96" rot="R90"/>
@@
 </segment>
 <segment>
-<pinref part="SJ2" gate="1" pin="2"/>
+<pinref part="U-SDA-5V" gate="1" pin="2"/>
 <wire x1="2.54" y1="88.9" x2="2.54" y2="91.44" width="0.1524" layer="91"/>
 <wire x1="2.54" y1="91.44" x2="10.16" y2="91.44" width="0.1524" layer="91"/>
-<pinref part="SJ1" gate="1" pin="2"/>
+<pinref part="U-SCL-5V" gate="1" pin="2"/>
 <wire x1="10.16" y1="91.44" x2="10.16" y2="88.9" width="0.1524" layer="91"/>
 <pinref part="P+3" gate="1" pin="+5V"/>
@@
 <segment>
 <pinref part="R2" gate="G$1" pin="2"/>
-<pinref part="SJ2" gate="1" pin="1"/>
+<pinref part="U-SDA-5V" gate="1" pin="1"/>
 <wire x1="2.54" y1="78.74" x2="2.54" y2="76.2" width="0.1524" layer="91"/>
 </segment>
@@
 <net name="N$18" class="0">
 <segment>
-<pinref part="SJ1" gate="1" pin="1"/>
+<pinref part="U-SCL-5V" gate="1" pin="1"/>
 <pinref part="R3" gate="G$1" pin="2"/>
 <wire x1="10.16" y1="78.74" x2="10.16" y2="76.2" width="0.1524" layer="91"/>
